File: Relay_Jacks.kicad_sch (KiCad schematic)
At the start: 13 parts, among them J1 4, J3 4, K1 IM05JR, Q1 DMN62D0U-7

Commit message: Schematic done?
Parts:
- removed WP2: SND, g-art:WirePad_H0.95mm_22-24AWG, symbol #gplm:art/ART-1001-0P95
- removed WP4: RTN, g-art:WirePad_H0.95mm_22-24AWG, symbol #gplm:art/ART-1001-0P95
- added R2: 1k, Resistor_SMD:R_0402_1005Metric, symbol #gplm:res/RES-2002-001K
- added R4: 330, Resistor_SMD:R_0402_1005Metric, symbol #gplm:res/RES-2002-330R
- added U6: TLP170AM, Package_SO:SO-4_4.4x3.9mm_P2.54mm, symbol #gplm:opt/OPT-0004-0001
Connections:
- net GNDA: now also U6.4
- net GNDD: now also U6.3
- net OUT: now also R2.2, U6.6; no longer K1.6
- new net: K1.6, R2.1
- new net: R4.1, U6.1
- new net MUTE: R4.2
Other:
- moved on the sheet: J3

Commit message: Committing uncommitted work, not sure what it was
Connections:
- net RLY_CL+: now reaches C8.1, D1.1 (K), JP1.2 (C), K1.1
Changed lines of the file:
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@@
+		)
+	)
+	(label "RLY_CL+"
+		(at 162.56 76.2 180)
+		(effects
+			(font
+				(size 1.27 1.27)
+			)
+			(justify right bottom)
 		)
 	)
