File: relay-bypass.kicad_pcb (KiCad board)
At the start: 2 copper layers, 35 parts, among them K1 IM05JR, Q1 DMN62D0U-7, U1 STM32C011F4Ux, U2 TPSM861257RDXR

Commit message: Committing uncommitted work, not sure what it was
Parts:
- removed D2: SMF4L9.0A, Diode_SMD:D_SOD-123F
- removed R3: 30k, Resistor_SMD:R_0402_1005Metric
- removed the REF** at (95.5, 45.3)
- removed the REF** at (101.2, 43.9)
- removed U2: TPSM861257RDXR, g-reg:QFN-FCMOD
- removed WP2: SND, g-art:WirePad_H0.95mm_22-24AWG
- removed WP4: RTN, g-art:WirePad_H0.95mm_22-24AWG
- added C11: 100n, Capacitor_SMD:C_0402_1005Metric, F.Cu at (59.0, 76.0)
- added C12: 100n, Capacitor_SMD:C_0402_1005Metric, F.Cu at (59.0, 78.0)
- added C13: 100n, Capacitor_SMD:C_0402_1005Metric, F.Cu at (124.0, 66.2)
- added C14: 1u, Capacitor_SMD:C_0805_2012Metric, F.Cu at (88.0, 105.2)
- added C15: 2.2u, Capacitor_SMD:C_1206_3216Metric, F.Cu at (102.0, 99.0)
- added D3: Red, LED_SMD:LED_0402_1005Metric, F.Cu at (115.8, 65.8)
- added D6: SMF4L9.0A, Diode_SMD:D_SOD-123F, F.Cu at (89.3, 109.8)
- added J1: 4, g-con:Amphenol_ACJM-MHDR(M), B.Cu at (84.5, 52.0)
- added J2: 8, Connector_JST:JST_SH_BM08B-SRSS-TB_1x08-1MP_P1.00mm_Vertical, F.Cu at (164.8, 146.5)
- added J3: 4, g-con:Amphenol_ACJM-MHDR(M), B.Cu at (115.5, 52.0)
- added J4: 3, g-con:BarrelJack_CUI_PJ-051A, B.Cu at (98.8, 56.0)
- added Q2: DMP3099L, Package_TO_SOT_SMD:SOT-23, F.Cu at (89.2, 100.8)
- added Q3: DMN62D0U-7, Package_TO_SOT_SMD:SOT-23, F.Cu at (137.6, 83.8)
- added R11: 1k, Resistor_SMD:R_0402_1005Metric, F.Cu at (56.2, 76.0)
- added R12: 1k, Resistor_SMD:R_0402_1005Metric, F.Cu at (56.2, 78.0)
- added R14: 3.3k, g-res:R_Axial_DIN0207_L6.3mm_D2.5mm_P7.5mm_Horizontal, F.Cu at (136.9, 87.8)
- added R15: 3.3k, Resistor_SMD:R_0603_1608Metric, F.Cu at (140.7, 87.8)
- added R16: 100k, Resistor_SMD:R_0402_1005Metric, F.Cu at (89.3, 96.2)
- added R19: 12k, Resistor_SMD:R_0402_1005Metric, F.Cu at (104.0, 104.0)
- added R20: 33k, Resistor_SMD:R_0402_1005Metric, F.Cu at (104.0, 106.0)
- added R8: 470, Resistor_SMD:R_0402_1005Metric, F.Cu at (113.5, 65.9)
- added REF**: SOT-223, Package_TO_SOT_SMD:SOT-223, F.Cu at (81.5, 87.5)
- added REF**: CP_Elec_5x5.8, Capacitor_SMD:CP_Elec_5x5.8, B.Cu at (126.8, 72.5)
- added TP4: PA8, g-art:TestPoint_PTH_H1.02mm_NoOutline, F.Cu at (65.8, 79.8)
- added TP5: PA3, g-art:TestPoint_PTH_H1.02mm_NoOutline, F.Cu at (65.8, 82.2)
- added U3: TLV76701DRVR, Package_SON:WSON-6-1EP_2x2mm_P0.65mm_EP1x1.6mm, F.Cu at (106.7, 98.8)
- added U6: TLP170AM, Package_SO:SO-4_4.4x3.9mm_P2.54mm, F.Cu at (109.8, 87.2)
- added WP10: LED+, g-art:WirePad_H0.95mm_22-24AWG, F.Cu at (141.9, 93.8)
- added WP11: +9V, g-art:WirePad_H0.95mm_22-24AWG, F.Cu at (103.8, 75.2)
- added WP12: GND, g-art:WirePad_H0.95mm_22-24AWG, F.Cu at (101.2, 75.2)
- added WP13: LED-, g-art:WirePad_H0.95mm_22-24AWG, F.Cu at (139.4, 93.8)
- added WP7: PA7, g-art:WirePad_H0.95mm_22-24AWG, F.Cu at (62.5, 82.5)
- added WP8: BYP, g-art:WirePad_H0.95mm_22-24AWG, F.Cu at (59.5, 82.5)
- added WP9: GND, g-art:WirePad_H0.95mm_22-24AWG, F.Cu at (56.5, 82.5)
- C1: value 22p -> 1u; footprint Capacitor_SMD:C_0402_1005Metric -> Capacitor_SMD:C_0603_1608Metric
- C10: value 1u -> 10p; footprint Capacitor_SMD:C_0805_2012Metric -> Capacitor_SMD:C_0402_1005Metric
- C2: value 22u -> 220n; footprint Capacitor_SMD:C_1206_3216Metric -> Capacitor_SMD:C_0402_1005Metric
- C3: value 100n -> 10n
- C4: value 100n -> 22n
- C5: value 10u -> 47u; footprint Capacitor_SMD:C_1210_3225Metric -> Capacitor_SMD:CP_Elec_6.3x5.8
- C6: value 4.7u -> 47u; footprint Capacitor_SMD:C_0805_2012Metric -> Capacitor_SMD:CP_Elec_6.3x5.8
- K1: moved to B.Cu
- R1: value 120k -> 1k
- R2: value 30k -> 1k
- R4: value 6.2k -> 330
- R6: value 4.7 -> 3.3
- TP1: value PG -> PA3; footprint TestPoint:TestPoint_Pad_D1.5mm -> g-art:TestPoint_PTH_H1.02mm_NoOutline
- WP1: value OUT -> RTN
- WP3: value IN -> SND
- WP5: value 9V -> 9VIN
- WP6: value 9V -> GND
- moved TP1 101.9 mm to (174.5, 136.2)
- moved JP3 54.2 mm to (79.5, 100.7)
- moved JP4 54.2 mm to (79.5, 104.2)
- moved C2 53.1 mm to (108.8, 103.5)
- moved C1 51.0 mm to (109.3, 106.2)
- moved C5 46.6 mm to (116.8, 102.2)
- moved R1 42.2 mm to (142.9, 83.8)
- moved C10 39.6 mm to (104.8, 95.0)
- moved C4 39.5 mm to (110.6, 98.8)
- moved C6 36.7 mm to (94.8, 87.0)
- moved R4 28.8 mm to (100.8, 88.2), turned to 90 degrees
- moved WP5 26.7 mm to (99.8, 34.8)
- moved WP6 26.6 mm to (102.2, 34.8)
- moved U1 25.1 mm to (119.1, 64.5)
- moved R2 24.3 mm to (104.5, 80.8)
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Connections:
- net Net-(D1-A) renamed /Relay_And_Jacks/RLY_CL-
- net Net-(D1-K) renamed /Relay_And_Jacks/RLY_CL+
- C1 pad 1: /3V Buck/VOUT -> +3.3V
- C1 pad 2: Net-(U2-FB) -> GNDD
- C10 pad 1: +9V -> +3.3V
- C10 pad 2: Net-(D2-A2) -> /FB
- C2 pad 1: /3V Buck/VOUT -> +3.3V
- C3 pad 1: /3V Buck/VOUT -> +3.3V
- C4 pad 1: +9V -> +3.3V
- C5 pad 1: +9V -> +3.3V
- C6 pad 1: +3.3V -> +9V
- C6 pad 2: GNDD -> GNDA
- JP3 pad 2: Net-(D2-A2) -> GND
- JP4 pad 2: Net-(D2-A2) -> GND
- K1 pad 3: /SEND -> /Relay_And_Jacks/SEND
- K1 pad 4: /IN -> /Relay_And_Jacks/IN
- K1 pad 5: /RETURN -> /Relay_And_Jacks/RETURN
- K1 pad 6: /OUT -> Net-(K1-Pad6)
- K1 pad 7: /IN -> /Relay_And_Jacks/IN
- R1 pad 1: /3V Buck/VOUT -> /LED_EXT
- R1 pad 2: Net-(U2-FB) -> Net-(Q3-G)
- R2 pad 1: Net-(U2-FB) -> Net-(K1-Pad6)
- R2 pad 2: GNDD -> /Relay_And_Jacks/OUT
- R4 pad 2: GNDD -> /MUTE
- TP1 pad 1: /3V Buck/PG -> /CLK_IN
- U1 pad 10: unconnected-(U1-PA5-Pad10) -> /RLY_SET
- U1 pad 13: /UART1_RX -> /SPR_PA8
- U1 pad 14: unconnected-(U1-PA9/PA11-Pad14) -> /LED_DBG
- U1 pad 15: unconnected-(U1-PA10/PA12-Pad15) -> /MUTE
- U1 pad 18: unconnected-(U1-PB6-Pad18) -> /SW_IN
- U1 pad 19: unconnected-(U1-PB7-Pad19) -> /SW_OUT
- U1 pad 20: unconnected-(U1-PC14-Pad20) -> /CLK_IN
- U1 pad 6: unconnected-(U1-PA1-Pad6) -> /UART1_RX
- U1 pad 8: unconnected-(U1-PA3-Pad8) -> /SPR_PA3
- U1 pad 9: /LED -> /LED_EXT
- WP1 pad 1: /OUT -> /Relay_And_Jacks/RETURN
- WP3 pad 1: /IN -> /Relay_And_Jacks/SEND
- WP5 pad 1: +9V -> +9VIN
- WP6 pad 1: Net-(D2-A2) -> GND
Other:
- board outline added: 59 x 25.8 mm
